File: mstd/io.kicad_sch (KiCad schematic)
At the start: 36 parts, among them Q2 2N7002, U10 74HCT05, U12 74HCT4066, U8 74HCT05

Commit message: Routing started
Parts:
- C17, C22, C23: footprint (none) -> Capacitor_SMD:C_0603_1608Metric_Pad1.08x0.95mm_HandSolder
- R10, R11, R12, R14, R15, R16, R17, R18, R19, R20, R21, R22, R23, R24, R25, R26, R27, R28, R29, R30, R31, R35, R36, R37, R38, R39: footprint (none) -> Resistor_SMD:R_0603_1608Metric_Pad0.98x0.95mm_HandSolder
- U10, U8: footprint (none) -> Package_SO:SO-14_3.9x8.65mm_P1.27mm
- X3: footprint (none) -> local:09722642801
- X4: footprint (none) -> local:snp15
Other:
- note added: "SWAP PIN ORDER!!! A/B01-32 <-> A/B32-0"
Changed lines of the file:
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@@
 		)
 	)
+	(text "SWAP PIN ORDER!!! A/B01-32 <-> A/B32-0"
+		(exclude_from_sim no)
+		(at 16.51 71.882 90)
+		(effects
+			(font
+				(size 1.27 1.27)
+			)
+		)
+	)
 	(hierarchical_label "ROM-CE3"
 		(shape output)
@@
 			)
 		)
-		(property "Footprint" ""
+		(property "Footprint" "Capacitor_SMD:C_0603_1608Metric_Pad1.08x0.95mm_HandSolder"
 			(at 90.4748 173.99 0)
 			(effects
@@
 			)
 		)
-		(property "Footprint" ""
+		(property "Footprint" "Resistor_SMD:R_0603_1608Metric_Pad0.98x0.95mm_HandSolder"
 			(at 260.35 42.672 90)
 			(effects
@@
 			)
 		)
-		(property "Footprint" ""
+		(property "Footprint" "Package_SO:SO-14_3.9x8.65mm_P1.27mm"
 			(at 243.84 50.8 0)
 			(effects
@@
 			)
 		)
-		(property "Footprint" ""
+		(property "Footprint" "Package_SO:SO-14_3.9x8.65mm_P1.27mm"
 			(at 31.75 180.34 0)
 			(effects
@@
 			)
 		)
-		(property "Footprint" ""
+		(property "Footprint" "local:09722642801"
 			(at 176.53 143.51 0)
 			(effects
@@
 			)
 		)
-		(property "Footprint" ""
+		(property "Footprint" "local:09722642801"
 			(at 90.17 41.91 0)
 			(effects
@@
 			)
 		)
-		(property "Footprint" ""
+		(property "Footprint" "Package_SO:SO-14_3.9x8.65mm_P1.27mm"
 			(at 91.44 129.54 0)
 			(effects
@@
 			)
 		)
-		(property "Footprint" ""
+		(property "Footprint" "Resistor_SMD:R_0603_1608Metric_Pad0.98x0.95mm_HandSolder"
 			(at 126.238 34.29 90)
 			(effects
@@
 			)
 		)
-		(property "Footprint" ""
+		(property "Footprint" "Resistor_SMD:R_0603_1608Metric_Pad0.98x0.95mm_HandSolder"
 			(at 114.3 128.778 90)
 			(effects
@@
 			)
 		)
-		(property "Footprint" ""
+		(property "Footprint" "Resistor_SMD:R_0603_1608Metric_Pad0.98x0.95mm_HandSolder"
 			(at 182.118 72.39 90)
 			(effects
@@
 			)
 		)
-		(property "Footprint" ""
+		(property "Footprint" "Resistor_SMD:R_0603_1608Metric_Pad0.98x0.95mm_HandSolder"
 			(at 114.3 145.288 90)
 			(effects
@@
 			)
 		)
-		(property "Footprint" ""
+		(property "Footprint" "local:09722642801"
 			(at 213.36 49.53 0)
 			(effects
@@
 			)
 		)
-		(property "Footprint" ""
+		(property "Footprint" "local:snp15"
 			(at 176.53 166.37 0)
 			(effects
@@
 			)
 		)
-		(property "Footprint" ""
+		(property "Footprint" "Resistor_SMD:R_0603_1608Metric_Pad0.98x0.95mm_HandSolder"
 			(at 123.698 34.29 90)
 			(effects
@@
 			)
 		)
-		(property "Footprint" ""
+		(property "Footprint" "Package_SO:SO-14_3.9x8.65mm_P1.27mm"
 			(at 139.7 48.26 0)
 			(effects
@@
 			)
 		)
-		(property "Footprint" ""
+		(property "Footprint" "Package_SO:SO-14_3.9x8.65mm_P1.27mm"
 			(at 60.96 180.34 0)
 			(effects
@@
 			)
 		)
-		(property "Footprint" ""
+		(property "Footprint" "Resistor_SMD:R_0603_1608Metric_Pad0.98x0.95mm_HandSolder"
 			(at 114.3 158.242 90)
 			(effects
@@
 			)
 		)
-		(property "Footprint" ""
+		(property "Footprint" "Resistor_SMD:R_0603_1608Metric_Pad0.98x0.95mm_HandSolder"
 			(at 177.038 72.39 90)
 			(effects
@@
 			)
 		)
-		(property "Footprint" ""
+		(property "Footprint" "Capacitor_SMD:C_0603_1608Metric_Pad1.08x0.95mm_HandSolder"
 			(at 81.5848 173.99 0)
 			(effects
@@
 			)
 		)
-		(property "Footprint" ""
+		(property "Footprint" "Package_SO:SO-14_3.9x8.65mm_P1.27mm"
 			(at 139.7 55.88 0)
 			(effects
@@
 			)
 		)
-		(property "Footprint" ""
+		(property "Footprint" "Package_SO:SO-14_3.9x8.65mm_P1.27mm"
 			(at 218.44 106.68 0)
 			(effects
@@
 			)
 		)
-		(property "Footprint" ""
+		(property "Footprint" "local:09722642801"
 			(at 111.76 113.03 0)
 			(effects
@@
 			)
 		)
-		(property "Footprint" ""
+		(property "Footprint" "Resistor_SMD:R_0603_1608Metric_Pad0.98x0.95mm_HandSolder"
 			(at 128.778 34.29 90)
 			(effects
@@
 			)
 		)
-		(property "Footprint" ""
+		(property "Footprint" "Resistor_SMD:R_0603_1608Metric_Pad0.98x0.95mm_HandSolder"
 			(at 249.682 111.76 90)
 			(effects
@@
 			)
 		)
-		(property "Footprint" ""
+		(property "Footprint" "Package_SO:SO-14_3.9x8.65mm_P1.27mm"
 			(at 91.44 138.43 0)
 			(effects
@@
 			)
 		)
-		(property "Footprint" ""
+		(property "Footprint" "local:snp15"
 			(at 44.45 41.91 0)
 			(effects
@@
 			)
 		)
-		(property "Footprint" ""
+		(property "Footprint" "Resistor_SMD:R_0603_1608Metric_Pad0.98x0.95mm_HandSolder"
 			(at 231.648 96.52 90)
 			(effects
@@
 			)
 		)
-		(property "Footprint" ""
+		(property "Footprint" "Resistor_SMD:R_0603_1608Metric_Pad0.98x0.95mm_HandSolder"
 			(at 129.54 83.058 90)
 			(effects
@@
 			)
 		)
-		(property "Footprint" ""
+		(property "Footprint" "Package_SO:SO-14_3.9x8.65mm_P1.27mm"
 			(at 207.01 135.89 0)
 			(effects
@@
 			)
 		)
-		(property "Footprint" ""
+		(property "Footprint" "Resistor_SMD:R_0603_1608Metric_Pad0.98x0.95mm_HandSolder"
 			(at 179.578 72.39 90)
 			(effects
@@
 			)
 		)
-		(property "Footprint" ""
+		(property "Footprint" "Resistor_SMD:R_0603_1608Metric_Pad0.98x0.95mm_HandSolder"
 			(at 150.368 33.02 90)
 			(effects
@@
 			)
 		)
-		(property "Footprint" ""
+		(property "Footprint" "Package_SO:SO-14_3.9x8.65mm_P1.27mm"
 			(at 91.44 162.56 0)
 			(effects
@@
 			)
 		)
-		(property "Footprint" ""
+		(property "Footprint" "Resistor_SMD:R_0603_1608Metric_Pad0.98x0.95mm_HandSolder"
 			(at 114.3 154.178 90)
 			(effects
@@
 			)
 		)
-		(property "Footprint" ""
+		(property "Footprint" "Package_SO:SO-14_3.9x8.65mm_P1.27mm"
 			(at 91.44 146.05 0)
 			(effects
@@
 			)
 		)
-		(property "Footprint" ""
+		(property "Footprint" "Package_SO:SO-14_3.9x8.65mm_P1.27mm"
 			(at 91.44 154.94 0)
 			(effects
@@
 			)
 		)
-		(property "Footprint" ""
+		(property "Footprint" "Resistor_SMD:R_0603_1608Metric_Pad0.98x0.95mm_HandSolder"
 			(at 141.478 185.42 90)
 			(effects
@@
 			)
 		)
-		(property "Footprint" ""
+		(property "Footprint" "Resistor_SMD:R_0603_1608Metric_Pad0.98x0.95mm_HandSolder"
 			(at 129.54 108.458 90)
 			(effects
@@
 			)
 		)
-		(property "Footprint" ""
+		(property "Footprint" "Resistor_SMD:R_0603_1608Metric_Pad0.98x0.95mm_HandSolder"
 			(at 200.152 115.57 90)
 			(effects
@@
 			)
 		)
-		(property "Footprint" ""
+		(property "Footprint" "Capacitor_SMD:C_0603_1608Metric_Pad1.08x0.95mm_HandSolder"
 			(at 72.6948 173.99 0)
 			(effects
@@
 			)
 		)
-		(property "Footprint" ""
+		(property "Footprint" "Resistor_SMD:R_0603_1608Metric_Pad0.98x0.95mm_HandSolder"
 			(at 114.3 137.668 90)
 			(effects
@@
 			)
 		)
-		(property "Footprint" ""
+		(property "Footprint" "local:09722642801"
 			(at 44.45 102.87 0)
 			(effects
@@
 			)
 		)
-		(property "Footprint" ""
+		(property "Footprint" "Resistor_SMD:R_0603_1608Metric_Pad0.98x0.95mm_HandSolder"
 			(at 251.968 143.51 90)
 			(effects
@@
 			)
 		)
-		(property "Footprint" ""
+		(property "Footprint" "Package_SO:SO-14_3.9x8.65mm_P1.27mm"
 			(at 229.87 125.73 0)
 			(effects
@@
 			)
 		)
-		(property "Footprint" ""
+		(property "Footprint" "Resistor_SMD:R_0603_1608Metric_Pad0.98x0.95mm_HandSolder"
 			(at 129.54 97.028 90)
 			(effects
@@
 			)
 		)
-		(property "Footprint" ""
+		(property "Footprint" "Resistor_SMD:R_0603_1608Metric_Pad0.98x0.95mm_HandSolder"
 			(at 256.54 24.638 90)
 			(effects
@@
 			)
 		)
-		(property "Footprint" ""
+		(property "Footprint" "Package_SO:SO-14_3.9x8.65mm_P1.27mm"
 			(at 139.7 40.64 0)
 			(effects
@@
 			)
 		)
-		(property "Footprint" ""
+		(property "Footprint" "Resistor_SMD:R_0603_1608Metric_Pad0.98x0.95mm_HandSolder"
 			(at 168.148 33.02 90)
 			(effects
@@
 			)
 		)
-		(property "Footprint" ""
+		(property "Footprint" "Resistor_SMD:R_0603_1608Metric_Pad0.98x0.95mm_HandSolder"
 			(at 202.692 152.4 90)
 			(effects
@@
 			)
 		)
-		(property "Footprint" ""
+		(property "Footprint" "local:snp15"
 			(at 213.36 68.58 0)
 			(effects
@@
 			)
 		)
-		(property "Footprint" ""
+		(property "Footprint" "local:snp15"
 			(at 44.45 165.1 0)
 			(effects
@@
 			)
 		)
-		(property "Footprint" ""
+		(property "Footprint" "Resistor_SMD:R_0603_1608Metric_Pad0.98x0.95mm_HandSolder"
 			(at 159.258 33.02 90)
 			(effects
@@
 			)
 		)
-		(property "Footprint" ""
+		(property "Footprint" "Resistor_SMD:R_0603_1608Metric_Pad0.98x0.95mm_HandSolder"
 			(at 260.35 28.448 90)
 			(effects
@@
 			)
 		)
-		(property "Footprint" ""
+		(property "Footprint" "local:snp15"
 			(at 115.57 66.04 0)
 			(effects

Commit message: Update Harting connector pin numeration to match SNP
Parts:
- X3: footprint local:09722642801 -> local:09722642801-1
Changed lines of the file:
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@@
 			)
 		)
-		(property "Footprint" "local:09722642801"
+		(property "Footprint" "local:09722642801-1"
 			(at 176.53 143.51 0)
 			(effects
@@
 			)
 		)
-		(property "Footprint" "local:09722642801"
+		(property "Footprint" "local:09722642801-1"
 			(at 90.17 41.91 0)
 			(effects
@@
 			)
 		)
-		(property "Footprint" "local:09722642801"
+		(property "Footprint" "local:09722642801-1"
 			(at 213.36 49.53 0)
 			(effects
@@
 			)
 		)
-		(property "Footprint" "local:09722642801"
+		(property "Footprint" "local:09722642801-1"
 			(at 111.76 113.03 0)
 			(effects
@@
 			)
 		)
-		(property "Footprint" "local:09722642801"
+		(property "Footprint" "local:09722642801-1"
 			(at 44.45 102.87 0)
 			(effects

Commit message: Routhing in finilizing stage
Parts:
- renumbered U8 to U10, U10 to U8
Connections:
- net DAL4: now also X4.B16 (DAL4); no longer X4.B28 (DAL4)
- net DOUT: now also U8.10; no longer U8.6
- net IAKN: now also U8.2; no longer U8.8
- net ROM-CE1: now also U10.8; no longer U10.10
- net RPLY: now also U8.9; no longer U8.3
- net S-BK: now also U8.6; no longer U8.12
- net SYNC: now also U8.12; no longer U8.2
- net WTB: now also U10.4; no longer U10.8
- net at X3.A24 (IAKN2), X4.A5 (IAKN): now also U8.1; no longer U8.9
- net at D4.2, R19.1, X3.B19 (INIT): now also U8.5; no longer U8.13
- net at X3.B22 (SINC), X4.A15 (SINC): now also U8.13; no longer U8.1
- net at R35.1, X4.B14 (CE1): now also U10.9; no longer U10.11
- net at X3.B20 (RPLY), X4.B15 (RPLY): now also U8.8; no longer U8.4
- net at X3.B21 (DOUT), X4.B8 (DOUT): now also U8.11; no longer U8.5
- net at X3.B11 (WTBT), X4.A8 (WTBT): now also U10.3; no longer U10.9
Other:
- note removed: "SWAP PIN ORDER!!! A/B01-32 <-> A/B32-0"
Changed lines of the file:
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@@
 		)
 	)
-	(text "SWAP PIN ORDER!!! A/B01-32 <-> A/B32-0"
-		(exclude_from_sim no)
-		(at 16.51 71.882 90)
-		(effects
-			(font
-				(size 1.27 1.27)
-			)
-		)
-	)
 	(hierarchical_label "ROM-CE3"
 		(shape output)
@@
 		(lib_id "local1:74HCT05")
 		(at 243.84 50.8 0)
-		(unit 4)
+		(unit 1)
 		(exclude_from_sim no)
 		(in_bom yes)
 		(on_board yes)
 		(dnp no)
-		(property "Reference" "U10"
+		(property "Reference" "U8"
 			(at 243.586 45.212 0)
 			(effects
@@
 			(project "mstd"
 				(path "/83a6c476-134a-4a4c-b05a-3c6f7ef5b0c5/c6989856-7d6c-495d-a92f-ca8859aec99b"
-					(reference "U10")
-					(unit 4)
+					(reference "U8")
+					(unit 1)
 				)
 			)
@@
 		(lib_id "local1:74HCT05")
 		(at 91.44 129.54 0)
-		(unit 1)
+		(unit 6)
 		(exclude_from_sim no)
 		(in_bom yes)
@@
 				(path "/83a6c476-134a-4a4c-b05a-3c6f7ef5b0c5/c6989856-7d6c-495d-a92f-ca8859aec99b"
 					(reference "U8")
-					(unit 1)
+					(unit 6)
 				)
 			)
@@
 		(dnp no)
 		(fields_autoplaced yes)
-		(property "Reference" "U8"
+		(property "Reference" "U10"
 			(at 139.7 39.37 0)
 			(effects
@@
 			(project "mstd"
 				(path "/83a6c476-134a-4a4c-b05a-3c6f7ef5b0c5/c6989856-7d6c-495d-a92f-ca8859aec99b"
-					(reference "U8")
+					(reference "U10")
 					(unit 6)
 				)
@@
 		(lib_id "local1:74HCT05")
 		(at 218.44 106.68 0)
-		(unit 6)
+		(unit 3)
 		(exclude_from_sim no)
 		(in_bom yes)
@@
 		(dnp no)
 		(fields_autoplaced yes)
-		(property "Reference" "U10"
+		(property "Reference" "U8"
 			(at 218.44 97.79 0)
 			(effects
@@
 			(project "mstd"
 				(path "/83a6c476-134a-4a4c-b05a-3c6f7ef5b0c5/c6989856-7d6c-495d-a92f-ca8859aec99b"
-					(reference "U10")
-					(unit 6)
+					(reference "U8")
+					(unit 3)
 				)
 			)
@@
 		(lib_id "local1:74HCT05")
 		(at 91.44 162.56 180)
-		(unit 2)
+		(unit 4)
 		(exclude_from_sim no)
 		(in_bom yes)
 		(on_board yes)
 		(dnp no)
-		(property "Reference" "U10"
+		(property "Reference" "U8"
 			(at 86.614 164.846 0)
 			(effects
@@
 			(project "mstd"
 				(path "/83a6c476-134a-4a4c-b05a-3c6f7ef5b0c5/c6989856-7d6c-495d-a92f-ca8859aec99b"
-					(reference "U10")
-					(unit 2)
+					(reference "U8")
+					(unit 4)
 				)
 			)
@@
 		(lib_id "local1:74HCT05")
 		(at 91.44 146.05 0)
-		(unit 3)
+		(unit 5)
 		(exclude_from_sim no)
 		(in_bom yes)
@@
 				(path "/83a6c476-134a-4a4c-b05a-3c6f7ef5b0c5/c6989856-7d6c-495d-a92f-ca8859aec99b"
 					(reference "U8")
-					(unit 3)
+					(unit 5)
 				)
 			)
@@
 		(lib_id "local1:74HCT05")
 		(at 91.44 154.94 0)
-		(unit 4)
+		(unit 2)
 		(exclude_from_sim no)
 		(in_bom yes)
 		(on_board yes)
 		(dnp no)
-		(fields_autoplaced yes)
-		(property "Reference" "U8"
-			(at 91.44 146.05 0)
+		(property "Reference" "U10"
+			(at 92.964 151.13 0)
 			(effects
 				(font
 					(size 1.27 1.27)
 				)
-				(hide yes)
 			)
 		)
@@
 			(project "mstd"
 				(path "/83a6c476-134a-4a4c-b05a-3c6f7ef5b0c5/c6989856-7d6c-495d-a92f-ca8859aec99b"
-					(reference "U8")
-					(unit 4)
+					(reference "U10")
+					(unit 2)
 				)
 			)
@@
 		(lib_id "local1:74HCT05")
 		(at 139.7 40.64 0)
-		(unit 5)
+		(unit 4)
 		(exclude_from_sim no)
 		(in_bom yes)
@@
 		(dnp no)
 		(fields_autoplaced yes)
-		(property "Reference" "U8"
+		(property "Reference" "U10"
 			(at 139.7 31.75 0)
 			(effects
@@
 			(project "mstd"
 				(path "/83a6c476-134a-4a4c-b05a-3c6f7ef5b0c5/c6989856-7d6c-495d-a92f-ca8859aec99b"
-					(reference "U8")
-					(unit 5)
+					(reference "U10")
+					(unit 4)
 				)
 			)
@@
 	)
 	(symbol
+		(lib_name "UKNC_SEP_1")
 		(lib_id "local1:UKNC_SEP")
 		(at 49.53 144.78 0)
@@
 		(pin "B22"
 		)
-		(pin "B28"
+		(pin "B16"
 		)
 		(pin "A12"
