File: mstd/pwr.kicad_sch (KiCad schematic)
At the start: 21 parts, among them J2 Barrel_Jack, Q1 SI2301CDS-T1-GE3, U1 ICE40UP5K-SG48ITR, U2 TLV70212DBVR, U3 TMI6050-33

Commit message: Routing started
Parts:
- C1, C10, C11, C2, C3, C4, C9: footprint (none) -> Capacitor_SMD:C_0603_1608Metric_Pad1.08x0.95mm_HandSolder
- C5, C6, C7: footprint (none) -> Capacitor_THT:CP_Radial_D5.0mm_P2.00mm
- C8: footprint (none) -> Capacitor_THT:CP_Radial_D6.3mm_P2.50mm
- J2: footprint (none) -> Connector_BarrelJack:BarrelJack_Wuerth_6941xx301002
- R1, R33, R34: footprint (none) -> Resistor_SMD:R_0603_1608Metric_Pad0.98x0.95mm_HandSolder
- X3: footprint (none) -> local:09722642801
- X4: footprint (none) -> local:snp15
Changed lines of the file:
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@@
 			)
 		)
-		(property "Footprint" ""
+		(property "Footprint" "Capacitor_THT:CP_Radial_D6.3mm_P2.50mm"
 			(at 44.45 64.77 0)
 			(effects
@@
 			)
 		)
-		(property "Footprint" ""
+		(property "Footprint" "Resistor_SMD:R_0603_1608Metric_Pad0.98x0.95mm_HandSolder"
 			(at 49.022 139.7 90)
 			(effects
@@
 			)
 		)
-		(property "Footprint" ""
+		(property "Footprint" "Capacitor_SMD:C_0603_1608Metric_Pad1.08x0.95mm_HandSolder"
 			(at 160.9852 46.99 0)
 			(effects
@@
 			)
 		)
-		(property "Footprint" ""
+		(property "Footprint" "Resistor_SMD:R_0603_1608Metric_Pad0.98x0.95mm_HandSolder"
 			(at 59.69 132.588 90)
 			(effects
@@
 			)
 		)
-		(property "Footprint" ""
+		(property "Footprint" "Capacitor_SMD:C_0603_1608Metric_Pad1.08x0.95mm_HandSolder"
 			(at 60.6552 67.31 0)
 			(effects
@@
 			)
 		)
-		(property "Footprint" ""
+		(property "Footprint" "Capacitor_SMD:C_0603_1608Metric_Pad1.08x0.95mm_HandSolder"
 			(at 153.3652 67.31 0)
 			(effects
@@
 			)
 		)
-		(property "Footprint" ""
+		(property "Footprint" "Capacitor_THT:CP_Radial_D5.0mm_P2.00mm"
 			(at 134.62 63.5 0)
 			(effects
@@
 			)
 		)
-		(property "Footprint" ""
+		(property "Footprint" "Connector_BarrelJack:BarrelJack_Wuerth_6941xx301002"
 			(at 31.75 122.936 0)
 			(effects
@@
 			)
 		)
-		(property "Footprint" ""
+		(property "Footprint" "Capacitor_THT:CP_Radial_D5.0mm_P2.00mm"
 			(at 181.61 86.36 0)
 			(effects
@@
 			)
 		)
-		(property "Footprint" ""
+		(property "Footprint" "Capacitor_SMD:C_0603_1608Metric_Pad1.08x0.95mm_HandSolder"
 			(at 102.5652 90.17 0)
 			(effects
@@
 			)
 		)
-		(property "Footprint" ""
+		(property "Footprint" "Resistor_SMD:R_0603_1608Metric_Pad0.98x0.95mm_HandSolder"
 			(at 139.7 56.388 90)
 			(effects
@@
 			)
 		)
-		(property "Footprint" ""
+		(property "Footprint" "local:snp15"
 			(at 124.46 181.61 0)
 			(effects
@@
 			)
 		)
-		(property "Footprint" ""
+		(property "Footprint" "local:09722642801"
 			(at 124.46 153.67 0)
 			(effects
@@
 			)
 		)
-		(property "Footprint" ""
+		(property "Footprint" "Capacitor_SMD:C_0603_1608Metric_Pad1.08x0.95mm_HandSolder"
 			(at 121.6152 67.31 0)
 			(effects
@@
 			)
 		)
-		(property "Footprint" ""
+		(property "Footprint" "Capacitor_THT:CP_Radial_D5.0mm_P2.00mm"
 			(at 146.05 44.45 0)
 			(effects
@@
 			)
 		)
-		(property "Footprint" ""
+		(property "Footprint" "Capacitor_SMD:C_0603_1608Metric_Pad1.08x0.95mm_HandSolder"
 			(at 168.6052 90.17 0)
 			(effects
@@
 			)
 		)
-		(property "Footprint" ""
+		(property "Footprint" "Capacitor_SMD:C_0603_1608Metric_Pad1.08x0.95mm_HandSolder"
 			(at 171.45 71.4248 0)
 			(effects

Commit message: Update Harting connector pin numeration to match SNP
Parts:
- X3: footprint local:09722642801 -> local:09722642801-1
Changed lines of the file:
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@@
 			)
 		)
-		(property "Footprint" "local:09722642801"
+		(property "Footprint" "local:09722642801-1"
 			(at 124.46 153.67 0)
 			(effects

Commit message: Routhing in finilizing stage
Parts:
- removed J2: Barrel_Jack, Connector_BarrelJack:BarrelJack_Wuerth_6941xx301002, symbol Connector:Barrel_Jack
- removed Q1: SI2301CDS-T1-GE3, easyeda2kicad:SOT-23-3_L3.0-W1.7-P0.95-LS2.9-BR, symbol EasyEDA:SI2301CDS-T1-GE3
- removed R33: 1K, Resistor_SMD:R_0603_1608Metric_Pad0.98x0.95mm_HandSolder, symbol Device:R
- removed R34: 100K, Resistor_SMD:R_0603_1608Metric_Pad0.98x0.95mm_HandSolder, symbol Device:R
- added R40, R41: 5K1, Resistor_SMD:R_0603_1608Metric_Pad0.98x0.95mm_HandSolder, symbol Device:R
- added USB1: TYPEC-306DDW-ARP16, easyeda2kicad:USB-C-TH_TYPEC-306DDW-ARP16, symbol EasyEDA:TYPEC-306DDW-ARP16
Connections:
- net +5V: now also USB1.A4 (VBUS), USB1.A9 (VBUS), USB1.B4 (VBUS), USB1.B9 (VBUS)
- net GND: now also R40.2, R41.2, USB1.17 (EH), USB1.18 (EH), USB1.19 (EH), USB1.20 (EH), USB1.A1 (GND), USB1.A12 (GND), USB1.B1 (GND), USB1.B12 (GND)
- new net: R41.1, USB1.B5 (CC2)
- new net: R40.1, USB1.A5 (CC1)
- no-connect marks 4 -> 6
